File: uefi2.kicad_sch (KiCad schematic)
At the start: 52 parts, among them J1 USB_B_Mini, J1 USB_C, J10 Conn_02x08_Odd_Even, J17 Conn_01x06, J2 Conn_02x10_Odd_Even, J3 Conn_02x03_Odd_Even, J4 Conn_02x04_Odd_Even, J5 Conn_01x05_Male, J5 Conn_02x09_Odd_Even, M1 Module-power_12and5V-0.2, M3 Module-knock-0.2, M3 Module-vr-discrete-0.5, M4 Module-vr-max9924-0.1, M5 Module-wbo-0.5, M6 Module:mega-mcu100/0.3, M7 Module-can-0.1, P1 Pad, P2 Pad, P3 Pad, P4 Pad, P7 Pad, P8 Pad, U4 JDY-33

Commit message: change revision from a to A0, change kicad file
Other:
- title: UAEFI -> UAEFI2
Changed lines of the file:
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@@
 	(paper "A3" portrait)
 	(title_block
-		(title "UAEFI")
-		(date "2024-03-27")
-		(rev "C")
+		(title "UAEFI2")
+		(date "2024-09-10")
+		(rev "A0")
 		(company "rusEFI.com")
 		(comment 1 "https://rusefi.com/s/uaefi")
